File: Buffered-Mult.kicad_sch (KiCad schematic)
At the start: 0 parts

Commit message: Initial schematic
Parts:
- added C1, C2, C3, C4, C5, C6: 100nF, symbol Device:C
- added D1, D2, D3, D4, D5, D6: LED, symbol Device:LED
- added J1: Eurorack PWR, symbol Connector_Generic:Conn_02x05_Odd_Even
- added J10: OUTPUT2-3, symbol Connector_Audio:AudioJack2_SwitchT
- added J11: OUTPUT3-1, symbol Connector_Audio:AudioJack2_SwitchT
- added J12: OUTPUT3-2, symbol Connector_Audio:AudioJack2_SwitchT
- added J13: OUTPUT3-3, symbol Connector_Audio:AudioJack2_SwitchT
- added J2: INPUT1, symbol Connector_Audio:AudioJack2_SwitchT
- added J3: INPUT2, symbol Connector_Audio:AudioJack2_SwitchT
- added J4: INPUT3, symbol Connector_Audio:AudioJack2_SwitchT
- added J5: OUTPUT1-1, symbol Connector_Audio:AudioJack2_SwitchT
- added J6: OUTPUT1-2, symbol Connector_Audio:AudioJack2_SwitchT
- added J7: OUTPUT1-3, symbol Connector_Audio:AudioJack2_SwitchT
- added J8: OUTPUT2-1, symbol Connector_Audio:AudioJack2_SwitchT
- added J9: OUTPUT2-2, symbol Connector_Audio:AudioJack2_SwitchT
- added R1, R2, R3: 100K, symbol Device:R
- added U1, U2, U3: TL074, symbol Amplifier_Operational:TL074
Connections:
- new net: D1.2 (A), D2.1 (K), U1.13 (-)
- new net: D1.1 (K), D2.2 (A), U1.14
- new net: D5.2 (A), D6.1 (K), U3.13 (-)
- new net: D5.1 (K), D6.2 (A), U3.14
- new net: D3.2 (A), D4.1 (K), U2.13 (-)
- new net: D3.1 (K), D4.2 (A), U2.14
- new net +12V: C1.1, C3.1, C5.1, J1.10 (Pin_10), J1.9 (Pin_9), U1.4 (V+), U2.4 (V+), U3.4 (V+)
- new net -12V: C2.2, C4.2, C6.2, J1.1 (Pin_1), J1.2 (Pin_2), U1.11 (V-), U2.11 (V-), U3.11 (V-)
- new net GND: C1.2, C2.1, C3.2, C4.1, C5.2, C6.1, J1.3 (Pin_3), J1.4 (Pin_4), J1.5 (Pin_5), J1.6 (Pin_6), J1.7 (Pin_7), J1.8 (Pin_8), J10.S, J11.S, J12.S, J13.S, J2.S, J2.TN, J3.S, J4.S, J5.S, J6.S, J7.S, J8.S, J9.S, R1.2, R2.2, R3.2
- new net INPUT1: J2.T, J3.TN, R1.1, U1.10 (+), U1.12 (+), U1.3 (+), U1.5 (+)
- new net INPUT2: J3.T, J4.TN, R2.1, U2.10 (+), U2.12 (+), U2.3 (+), U2.5 (+)
- new net INPUT3: J4.T, R3.1, U3.10 (+), U3.12 (+), U3.3 (+), U3.5 (+)
- new net OUTPUT1-1: J5.T, U1.1, U1.2 (-)
- new net OUTPUT1-2: J6.T, U1.6 (-), U1.7
- new net OUTPUT1-3: J7.T, U1.8, U1.9 (-)
- new net OUTPUT2-1: J8.T, U2.1, U2.2 (-)
- new net OUTPUT2-2: J9.T, U2.6 (-), U2.7
- new net OUTPUT2-3: J10.T, U2.8, U2.9 (-)
- new net OUTPUT3-1: J11.T, U3.1, U3.2 (-)
- new net OUTPUT3-2: J12.T, U3.6 (-), U3.7
- new net OUTPUT3-3: J13.T, U3.8, U3.9 (-)
- no-connect marks 0 -> 9

Commit message: Updated schematic
Parts:
- added C10, C11, C9: 100pF, symbol Device:C
- added C7, C8: 10uF/25V, symbol Device:C_Polarized
- added D7, D8: D_Schottky, symbol Device:D_Schottky
- added R10, R11, R12, R13, R14, R15, R16, R17, R18, R4, R5, R6, R7, R8, R9: 1k, symbol Device:R
Connections:
- net +12V: now also C7.1, D7.1 (K); no longer J1.10 (Pin_10), J1.9 (Pin_9)
- net -12V: now also C8.2, D8.2 (A); no longer J1.1 (Pin_1), J1.2 (Pin_2)
- net GND: now also C10.2, C11.2, C7.2, C8.1, C9.2, R4.2, R5.2, R6.2
- net INPUT1: now also C9.1, R16.2; no longer J2.T, J3.TN, R1.1
- net INPUT2: now also C10.1, R17.2; no longer J3.T, J4.TN, R2.1
- net INPUT3: now also C11.1, R18.2; no longer J4.T, R3.1
- net OUTPUT1-1: now also R7.1; no longer U1.1
- net OUTPUT1-2: now also R8.1; no longer U1.7
- net OUTPUT1-3: now also R9.1; no longer U1.8
- net OUTPUT2-1: now also R10.1; no longer U2.1
- net OUTPUT2-2: now also R11.1; no longer U2.7
- net OUTPUT2-3: now also R12.1; no longer U2.8
- net OUTPUT3-1: now also R13.1; no longer U3.1
- net OUTPUT3-2: now also R14.1; no longer U3.7
- net OUTPUT3-3: now also R15.1; no longer U3.8
- net at D1.2 (A), D2.1 (K), U1.13 (-): now also R4.1
- net at D5.2 (A), D6.1 (K), U3.13 (-): now also R6.1
- net at D3.2 (A), D4.1 (K), U2.13 (-): now also R5.1
- new net: R8.2, U1.7
- new net: R12.2, U2.8
- new net: R11.2, U2.7
- new net: D8.1 (K), J1.1 (Pin_1), J1.2 (Pin_2)
- new net: D7.2 (A), J1.10 (Pin_10), J1.9 (Pin_9)
- new net: R7.2, U1.1
- new net: R10.2, U2.1
- new net: J2.T, J3.TN, R1.1, R16.1
- new net: R15.2, U3.8
- new net: J3.T, J4.TN, R17.1, R2.1
- new net: R9.2, U1.8
- new net: R13.2, U3.1
- new net: J4.T, R18.1, R3.1
- new net: R14.2, U3.7
Other:
- moved on the sheet: D1, D5, D6, J3, J4, R2, R3, U3A

Commit message: Updated schematic
Connections:
- net OUTPUT1-1: no longer U1.2 (-)
- net OUTPUT1-2: no longer U1.6 (-)
- net OUTPUT1-3: no longer U1.9 (-)
- net OUTPUT2-1: no longer U2.2 (-)
- net OUTPUT2-2: no longer U2.6 (-)
- net OUTPUT2-3: no longer U2.9 (-)
- net OUTPUT3-1: now also R13.2; no longer R13.1, U3.2 (-)
- net OUTPUT3-2: no longer U3.6 (-)
- net OUTPUT3-3: no longer U3.9 (-)
- net at R8.2, U1.7: now also U1.6 (-)
- net at R12.2, U2.8: now also U2.9 (-)
- net at R11.2, U2.7: now also U2.6 (-)
- net at R7.2, U1.1: now also U1.2 (-)
- net at R10.2, U2.1: now also U2.2 (-)
- net at R15.2, U3.8: now also U3.9 (-)
- net at R9.2, U1.8: now also U1.9 (-)
- net at U3.1: now also R13.1, U3.2 (-); no longer R13.2
- net at R14.2, U3.7: now also U3.6 (-)
Other:
- moved on the sheet: C10, C11, C9, D1, D2, D3, D4, D5, D6, J10, J11, J12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

Commit message: Add LCSC Part numbers
Parts:
- C1, C2, C3, C4, C5, C6: footprint (none) -> Capacitor_SMD:C_0603_1608Metric_Pad1.08x0.95mm_HandSolder; LCSC (none) -> C14663
- C10, C11, C9: footprint (none) -> Capacitor_SMD:C_0603_1608Metric_Pad1.08x0.95mm_HandSolder; LCSC (none) -> C14858
- C7, C8: footprint (none) -> Capacitor_SMD:CP_Elec_5x3; LCSC (none) -> C46550416
- D1, D2, D3, D4, D5, D6: footprint (none) -> LED_THT:LED_D3.0mm_FlatTop
- D7, D8: footprint (none) -> Diode_SMD:D_SOD-323; LCSC (none) -> C2480
- J1: footprint (none) -> Connector_IDC:IDC-Header_2x05_P2.54mm_Vertical
- J10, J11, J12, J13, J2, J3, J4, J5, J6, J7, J8, J9: footprint (none) -> Connector_Audio:Jack_3.5mm_QingPu_WQP-PJ398SM_Vertical_CircularHoles
- R1, R2, R3: footprint (none) -> Resistor_SMD:R_0603_1608Metric_Pad0.98x0.95mm_HandSolder; LCSC (none) -> C25803
- R10, R11, R12, R13, R14, R15, R16, R17, R18, R4, R5, R6, R7, R8, R9: footprint (none) -> Resistor_SMD:R_0603_1608Metric_Pad0.98x0.95mm_HandSolder; LCSC (none) -> C21190
- U1, U2, U3: footprint (none) -> Package_SO:SOIC-14_3.9x8.7mm_P1.27mm; LCSC (none) -> C2878713

Commit message: First draft of PCB
Parts:
- C7, C8: footprint Capacitor_SMD:CP_Elec_5x3 -> Capacitor_SMD:CP_Elec_5x5.4
- D7, D8: footprint Diode_SMD:D_SOD-323 -> Diode_SMD:D_SMA_Handsoldering
