File: Buffered-Mult.kicad_pcb (KiCad board)
At the start: 2 copper layers, 53 parts, among them J1 Eurorack PWR, J10 OUTPUT2-3, J11 OUTPUT3-1, J12 OUTPUT3-2, J13 OUTPUT3-3, J2 INPUT1, J3 INPUT2, J4 INPUT3, J5 OUTPUT1-1, J6 OUTPUT1-2, J7 OUTPUT1-3, J8 OUTPUT2-1, J9 OUTPUT2-2, U1 TL074, U2 TL074, U3 TL074

Commit message: First draft of PCB
Parts:
- C7, C8: footprint Capacitor_SMD:CP_Elec_5x3 -> Capacitor_SMD:CP_Elec_5x5.4
- D1, D2, D3, D4, D5, D6, J10, J11, J12, J13, J2, J3, J4, J5, J6, J7, J8, J9: moved to B.Cu
- D7, D8: footprint Diode_SMD:D_SOD-323 -> Diode_SMD:D_SMA_Handsoldering
- moved J1 110.8 mm to (37.5, 132.0), turned to 180 degrees
- moved R4 98.8 mm to (45.5, 37.3), turned to -90 degrees
- moved C1 96.9 mm to (33.8, 37.4), turned to -90 degrees
- moved R9 93.7 mm to (42.5, 51.1), turned to 180 degrees
- moved R16 92.8 mm to (49.7, 48.1)
- moved R7 92.6 mm to (42.6, 48.1), turned to 180 degrees
- moved C2 90.3 mm to (43.8, 37.3), turned to 90 degrees
- moved R8 89.3 mm to (46.1, 51.1), turned to 180 degrees
- moved R1 87.1 mm to (46.2, 48.1), turned to 180 degrees
- moved R13 86.8 mm to (42.5, 105.6)
- moved R15 86.5 mm to (42.5, 109.3), turned to 180 degrees
- moved C3 86.4 mm to (34.1, 64.9), turned to -90 degrees
- moved R12 85.0 mm to (42.4, 80.2), turned to 180 degrees
- moved C9 85.0 mm to (49.6, 51.1), turned to 180 degrees
- moved R10 84.5 mm to (42.5, 76.7), turned to 180 degrees
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Routing:
- net -12V: track 0.00 -> 155.0 mm, vias 0 -> 6
- net +12V: track 0.00 -> 116.7 mm, vias 0 -> 6
- net Net-(J2-PadT): track 0.00 -> 33.4 mm, vias 0 -> 1
- net Net-(J3-PadT): track 0.00 -> 33.4 mm, vias 0 -> 1
- net INPUT3: track 0.00 -> 31.5 mm
- net INPUT2: track 0.00 -> 31.3 mm
- net INPUT1: track 0.00 -> 29.9 mm
- net Net-(D3-K): track 0.00 -> 25.9 mm
- net Net-(D5-K): track 0.00 -> 25.7 mm
- net Net-(D1-K): track 0.00 -> 25.5 mm
- net Net-(U2A--): track 0.00 -> 22.0 mm
- net Net-(U3A--): track 0.00 -> 21.8 mm
- net Net-(U1A--): track 0.00 -> 21.3 mm
- net Net-(U3B--): track 0.00 -> 17.3 mm
- net Net-(U2B--): track 0.00 -> 17.2 mm
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- added copper zone on B.Cu, net GND
- added copper zone on F.Cu, net GND
Other:
- board outline added: 30 x 110 mm
- board text added: "Red Stripe"

Commit message: First cut of production files
Other:
- board text added: "JLCJLCJLCJLC"

Commit message: Second cut of production files
Other:
- board text removed: "JLCJLCJLCJLC"
Changed lines of the file:
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@@
+	)
+	(gr_rect
+		(start 52.5 132.5)
+		(end 57.5 137.5)
+		(stroke
+			(width 0.1)
+			(type solid)
+		)
+		(fill yes)
+		(layer "B.SilkS")
 	)
 	(gr_rect
@@
 		)
 	)
-	(gr_text "JLCJLCJLCJLC"
-		(at 59.4 139.4 0)
-		(layer "B.SilkS")
-		(effects
-			(font
-				(size 1.5 1.5)
-				(thickness 0.1)
-			)
-			(justify left bottom mirror)
-		)
-	)
