File: faceplate/Faceplate.kicad_pcb (KiCad board)
At the start: 2 copper layers, 30 x 128.5 mm, 22 parts

Commit message: Adding stuff to faceplate
Parts:
- H1, H10, H2, H9: footprint MountingHole:MountingHole_3.2mm_M3_Pad -> ModularHoles:Eurorack_Mounting_Slot_M3_Earthed
- moved H9 173.5 mm to (52.5, 33.0)
- moved H1 168.7 mm to (37.5, 33.0)
- moved H7 164.6 mm to (35.8, 104.2)
- moved H2 162.0 mm to (37.5, 155.5)
- moved H8 159.5 mm to (41.3, 104.2)
- moved H10 149.7 mm to (52.5, 155.5)
Other:
- board text added: "IN"
- board text added: "OUT"

Commit message: Add labels and group separators
Other:
- board text added: "Buffered Mult"

Commit message: Add artwork
Other:
- board text added: "+"
- board text added: "-"
- board text added: "TL074"

Commit message: Faceplate manufacturing files
Parts:
- H3, H4, H5, H6, H7, H8: footprint MountingHole:MountingHole_3.2mm_M3 -> ModularHoles:LED_3.2mm_M3
Changed lines of the file:
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@@
 		(sheetname "/")
 		(sheetfile "Faceplate.kicad_sch")
+		(units
+			(unit
+				(name "A")
+				(pins "1")
+			)
+		)
 		(attr exclude_from_bom)
 		(duplicate_pad_numbers_are_jumpers no)
@@
 		(sheetname "/")
 		(sheetfile "Faceplate.kicad_sch")
+		(units
+			(unit
+				(name "A")
+				(pins "1")
+			)
+		)
 		(attr exclude_from_bom)
 		(duplicate_pad_numbers_are_jumpers no)
@@
 		(embedded_fonts no)
 	)
-	(footprint "MountingHole:MountingHole_3.2mm_M3"
+	(footprint "ModularHoles:LED_3.2mm_M3"
 		(layer "F.Cu")
 		(at 35.77 46.25)
@@
 		(sheetname "/")
 		(sheetfile "Faceplate.kicad_sch")
+		(units
+			(unit
+				(name "A")
+				(pins)
+			)
+		)
 		(attr exclude_from_bom)
 		(duplicate_pad_numbers_are_jumpers no)
 		(fp_circle
 			(center 0 0)
-			(end 3.2 0)
+			(end 1.7 0)
 			(stroke
 				(width 0.15)
@@
 		(fp_circle
 			(center 0 0)
-			(end 3.45 0)
+			(end 1.8 0)
 			(stroke
 				(width 0.05)
@@
 		(embedded_fonts no)
 	)
-	(footprint "MountingHole:MountingHole_3.2mm_M3"
+	(footprint "ModularHoles:LED_3.2mm_M3"
 		(layer "F.Cu")
 		(at 35.77 104.25)
@@
 		(sheetname "/")
 		(sheetfile "Faceplate.kicad_sch")
+		(units
+			(unit
+				(name "A")
+				(pins)
+			)
+		)
 		(attr exclude_from_bom)
 		(duplicate_pad_numbers_are_jumpers no)
 		(fp_circle
 			(center 0 0)
-			(end 3.2 0)
+			(end 1.7 0)
 			(stroke
 				(width 0.15)
@@
 		(fp_circle
 			(center 0 0)
-			(end 3.45 0)
+			(end 1.8 0)
 			(stroke
 				(width 0.05)
@@
 		(sheetname "/")
 		(sheetfile "Faceplate.kicad_sch")
+		(units
+			(unit
+				(name "A")
+				(pins "1")
+			)
+		)
 		(attr exclude_from_bom)
 		(duplicate_pad_numbers_are_jumpers no)
@@
 		(sheetname "/")
 		(sheetfile "Faceplate.kicad_sch")
+		(units
+			(unit
+				(name "A")
+				(pins "1")
+			)
+		)
 		(attr exclude_from_bom)
 		(duplicate_pad_numbers_are_jumpers no)
@@
 		(sheetname "/")
 		(sheetfile "Faceplate.kicad_sch")
+		(units
+			(unit
+				(name "A")
+				(pins "1")
+			)
+		)
 		(attr smd exclude_from_bom)
 		(duplicate_pad_numbers_are_jumpers no)
@@
 		(sheetname "/")
 		(sheetfile "Faceplate.kicad_sch")
+		(units
+			(unit
+				(name "A")
+				(pins "1")
+			)
+		)
 		(attr exclude_from_bom)
 		(duplicate_pad_numbers_are_jumpers no)
@@
 		(sheetname "/")
 		(sheetfile "Faceplate.kicad_sch")
+		(units
+			(unit
+				(name "A")
+				(pins "1")
+			)
+		)
 		(attr smd exclude_from_bom)
 		(duplicate_pad_numbers_are_jumpers no)
@@
 		(sheetname "/")
 		(sheetfile "Faceplate.kicad_sch")
+		(units
+			(unit
+				(name "A")
+				(pins "1")
+			)
+		)
 		(attr exclude_from_bom)
 		(duplicate_pad_numbers_are_jumpers no)
@@
 		(sheetname "/")
 		(sheetfile "Faceplate.kicad_sch")
+		(units
+			(unit
+				(name "A")
+				(pins "1")
+			)
+		)
 		(attr exclude_from_bom)
 		(duplicate_pad_numbers_are_jumpers no)
@@
 		(sheetname "/")
 		(sheetfile "Faceplate.kicad_sch")
+		(units
+			(unit
+				(name "A")
+				(pins "1")
+			)
+		)
 		(attr exclude_from_bom)
 		(duplicate_pad_numbers_are_jumpers no)
@@
 		(sheetname "/")
 		(sheetfile "Faceplate.kicad_sch")
+		(units
+			(unit
+				(name "A")
+				(pins "1")
+			)
+		)
 		(attr exclude_from_bom)
 		(duplicate_pad_numbers_are_jumpers no)
@@
 		(embedded_fonts no)
 	)
-	(footprint "MountingHole:MountingHole_3.2mm_M3"
+	(footprint "ModularHoles:LED_3.2mm_M3"
 		(layer "F.Cu")
 		(at 35.77 75.25)
@@
 		(sheetname "/")
 		(sheetfile "Faceplate.kicad_sch")
+		(units
+			(unit
+				(name "A")
+				(pins)
+			)
+		)
 		(attr exclude_from_bom)
 		(duplicate_pad_numbers_are_jumpers no)
 		(fp_circle
 			(center 0 0)
-			(end 3.2 0)
+			(end 1.7 0)
 			(stroke
 				(width 0.15)
@@
 		(fp_circle
 			(center 0 0)
-			(end 3.45 0)
+			(end 1.8 0)
 			(stroke
 				(width 0.05)
@@
 		(sheetname "/")
 		(sheetfile "Faceplate.kicad_sch")
+		(units
+			(unit
+				(name "A")
+				(pins "1")
+			)
+		)
 		(attr exclude_from_bom)
 		(duplicate_pad_numbers_are_jumpers no)
@@
 		(embedded_fonts no)
 	)
-	(footprint "MountingHole:MountingHole_3.2mm_M3"
+	(footprint "ModularHoles:LED_3.2mm_M3"
 		(layer "F.Cu")
 		(at 41.27 104.25)
@@
 		(sheetname "/")
 		(sheetfile "Faceplate.kicad_sch")
+		(units
+			(unit
+				(name "A")
+				(pins)
+			)
+		)
 		(attr exclude_from_bom)
 		(duplicate_pad_numbers_are_jumpers no)
 		(fp_circle
 			(center 0 0)
-			(end 3.2 0)
+			(end 1.7 0)
 			(stroke
 				(width 0.15)
@@
 		(fp_circle
 			(center 0 0)
-			(end 3.45 0)
+			(end 1.8 0)
 			(stroke
 				(width 0.05)
@@
 		(sheetname "/")
 		(sheetfile "Faceplate.kicad_sch")
+		(units
+			(unit
+				(name "A")
+				(pins "1")
+			)
+		)
 		(attr smd exclude_from_bom)
 		(duplicate_pad_numbers_are_jumpers no)
@@
 		(sheetname "/")
 		(sheetfile "Faceplate.kicad_sch")
+		(units
+			(unit
+				(name "A")
+				(pins "1")
+			)
+		)
 		(attr exclude_from_bom)
 		(duplicate_pad_numbers_are_jumpers no)
@@
 		(embedded_fonts no)
 	)
-	(footprint "MountingHole:MountingHole_3.2mm_M3"
+	(footprint "ModularHoles:LED_3.2mm_M3"
 		(layer "F.Cu")
 		(at 41.27 75.25)
@@
 		(sheetname "/")
 		(sheetfile "Faceplate.kicad_sch")
+		(units
+			(unit
+				(name "A")
+				(pins)
+			)
+		)
 		(attr exclude_from_bom)
 		(duplicate_pad_numbers_are_jumpers no)
 		(fp_circle
 			(center 0 0)
-			(end 3.2 0)
+			(end 1.7 0)
 			(stroke
 				(width 0.15)
@@
 		(fp_circle
 			(center 0 0)
-			(end 3.45 0)
+			(end 1.8 0)
 			(stroke
 				(width 0.05)
@@
 		(sheetname "/")
 		(sheetfile "Faceplate.kicad_sch")
+		(units
+			(unit
+				(name "A")
+				(pins "1")
+			)
+		)
 		(attr smd exclude_from_bom)
 		(duplicate_pad_numbers_are_jumpers no)
@@
 		(embedded_fonts no)
 	)
-	(footprint "MountingHole:MountingHole_3.2mm_M3"
+	(footprint "ModularHoles:LED_3.2mm_M3"
 		(layer "F.Cu")
 		(at 41.27 46.25)
@@
 		(sheetname "/")
 		(sheetfile "Faceplate.kicad_sch")
+		(units
+			(unit
+				(name "A")
+				(pins)
+			)
+		)
 		(attr exclude_from_bom)
 		(duplicate_pad_numbers_are_jumpers no)
 		(fp_circle
 			(center 0 0)
-			(end 3.2 0)
+			(end 1.7 0)
 			(stroke
 				(width 0.15)
@@
 		(fp_circle
 			(center 0 0)
-			(end 3.45 0)
+			(end 1.8 0)
 			(stroke
 				(width 0.05)
@@
 		(sheetname "/")
 		(sheetfile "Faceplate.kicad_sch")
+		(units
+			(unit
+				(name "A")
+				(pins "1")
+			)
+		)
 		(attr exclude_from_bom)
 		(duplicate_pad_numbers_are_jumpers no)
@@
 		(end 38.048471 133.954236)
 		(stroke
-			(width 0)
+			(width 0.1)
 			(type solid)
 		)
@@
 		(end 38.048471 136.26949)
 		(stroke
-			(width 0)
+			(width 0.1)
 			(type solid)
 		)
@@
 		(end 38.048471 138.584746)
 		(stroke
-			(width 0)
+			(width 0.1)
 			(type solid)
 		)
@@
 		(end 38.048471 140.900001)
 		(stroke
-			(width 0)
+			(width 0.1)
 			(type solid)
 		)
@@
 		(end 38.048471 143.215253)
 		(stroke
-			(width 0)
+			(width 0.1)
 			(type solid)
 		)
@@
 		(end 38.048471 145.53051)
 		(stroke
-			(width 0)
+			(width 0.1)
 			(type solid)
 		)
@@
 		(end 38.048471 147.845763)
 		(stroke
-			(width 0)
+			(width 0.1)
 			(type solid)
 		)
@@
 		(end 54.37102 133.954236)
 		(stroke
-			(width 0)
+			(width 0.1)
 			(type solid)
 		)
@@
 		(end 54.37102 136.26949)
 		(stroke
-			(width 0)
+			(width 0.1)
 			(type solid)
 		)
@@
 		(end 54.37102 138.584746)
 		(stroke
-			(width 0)
+			(width 0.1)
 			(type solid)
 		)
@@
 		(end 54.37102 140.900001)
 		(stroke
-			(width 0)
+			(width 0.1)
 			(type solid)
 		)
@@
 		(end 54.37102 143.215253)
 		(stroke
-			(width 0)
+			(width 0.1)
 			(type solid)
 		)
@@
 		(end 54.37102 145.53051)
 		(stroke
-			(width 0)
+			(width 0.1)
 			(type solid)
 		)
@@
 		(end 54.37102 147.845763)
 		(stroke
-			(width 0)
-			(type solid)
-		)
+			(width 0.1)
+			(type solid)
+		)
