File: faceplate/Faceplate.kicad_sch (KiCad schematic)
At the start: 22 parts

Commit message: Adding stuff to faceplate
Parts:
- H1, H10, H2, H9: footprint MountingHole:MountingHole_3.2mm_M3_Pad -> ModularHoles:Eurorack_Mounting_Slot_M3_Earthed
Changed lines of the file:
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@@
 			)
 		)
-		(property "Footprint" "MountingHole:MountingHole_3.2mm_M3_Pad"
+		(property "Footprint" "ModularHoles:Eurorack_Mounting_Slot_M3_Earthed"
 			(at 43.18 85.09 0)
 			(hide yes)
@@
 			)
 		)
-		(property "Footprint" "MountingHole:MountingHole_3.2mm_M3_Pad"
+		(property "Footprint" "ModularHoles:Eurorack_Mounting_Slot_M3_Earthed"
 			(at 43.18 92.71 0)
 			(hide yes)
@@
 			)
 		)
-		(property "Footprint" "MountingHole:MountingHole_3.2mm_M3_Pad"
+		(property "Footprint" "ModularHoles:Eurorack_Mounting_Slot_M3_Earthed"
 			(at 82.55 85.09 0)
 			(hide yes)
@@
 			)
 		)
-		(property "Footprint" "MountingHole:MountingHole_3.2mm_M3_Pad"
+		(property "Footprint" "ModularHoles:Eurorack_Mounting_Slot_M3_Earthed"
 			(at 82.55 92.71 0)
 			(hide yes)

Commit message: Faceplate manufacturing files
Parts:
- H3, H4, H5, H6, H7, H8: footprint MountingHole:MountingHole_3.2mm_M3 -> ModularHoles:LED_3.2mm_M3
Changed lines of the file:
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@@
 			)
 		)
-		(property "Footprint" "MountingHole:MountingHole_3.2mm_M3"
+		(property "Footprint" "ModularHoles:LED_3.2mm_M3"
 			(at 40.64 34.29 0)
 			(hide yes)
@@
 			)
 		)
-		(property "Footprint" "MountingHole:MountingHole_3.2mm_M3"
+		(property "Footprint" "ModularHoles:LED_3.2mm_M3"
 			(at 40.5966 68.3641 0)
 			(hide yes)
@@
 			)
 		)
-		(property "Footprint" "MountingHole:MountingHole_3.2mm_M3"
+		(property "Footprint" "ModularHoles:LED_3.2mm_M3"
 			(at 40.64 60.96 0)
 			(hide yes)
@@
 			)
 		)
-		(property "Footprint" "MountingHole:MountingHole_3.2mm_M3"
+		(property "Footprint" "ModularHoles:LED_3.2mm_M3"
 			(at 40.64 53.34 0)
 			(hide yes)
@@
 			)
 		)
-		(property "Footprint" "MountingHole:MountingHole_3.2mm_M3"
+		(property "Footprint" "ModularHoles:LED_3.2mm_M3"
 			(at 40.64 40.64 0)
 			(hide yes)
@@
 			)
 		)
-		(property "Footprint" "MountingHole:MountingHole_3.2mm_M3"
+		(property "Footprint" "ModularHoles:LED_3.2mm_M3"
 			(at 40.64 46.99 0)
 			(hide yes)
